File: splitkb.kicad_pcb (KiCad board)
At the start: 2 copper layers, 166.4 x 132.1 mm, 145 parts, among them J1 MJ-4PP-9, K1 KEYSW, SW1 SW_PUSH, SW10 SW_PUSH, SW11 SW_PUSH, SW12 SW_PUSH, SW13 SW_PUSH, SW14 SW_PUSH, SW15 SW_PUSH, SW16 SW_PUSH, SW17 SW_PUSH, SW18 SW_PUSH, SW19 SW_PUSH, SW2 SW_PUSH, SW20 SW_PUSH, SW21 SW_PUSH, SW22 SW_PUSH, SW23 SW_PUSH, SW24 SW_PUSH, SW25 SW_PUSH, SW26 SW_PUSH, SW27 SW_PUSH, SW28 SW_PUSH, SW29 SW_PUSH, SW3 SW_PUSH, SW30 SW_PUSH, SW31 SW_PUSH, SW32 SW_PUSH, SW33 SW_PUSH, SW34 SW_PUSH, SW35 SW_PUSH, SW4 SW_PUSH, SW5 SW_PUSH, SW6 SW_PUSH, SW7 SW_PUSH, SW8 SW_PUSH, SW9 SW_PUSH, U1 ProMicro

Commit message: added holes
Parts:
- added REF**: MountingHole_4.3mm_M4_ISO14580, MountingHole:MountingHole_4.3mm_M4_ISO14580, F.Cu at (37.5, 117.5)
- added REF**: MountingHole_4.3mm_M4_ISO14580, MountingHole:MountingHole_4.3mm_M4_ISO14580, F.Cu at (37.5, 60.3)
- added REF**: MountingHole_4.3mm_M4_ISO14580, MountingHole:MountingHole_4.3mm_M4_ISO14580, F.Cu at (94.0, 90.8)
- added REF**: MountingHole_4.3mm_M4_ISO14580, MountingHole:MountingHole_4.3mm_M4_ISO14580, F.Cu at (94.0, 52.7)
- added REF**: MountingHole_4.3mm_M4_ISO14580, MountingHole:MountingHole_4.3mm_M4_ISO14580, F.Cu at (132.1, 61.0)
- added REF**: MountingHole_4.3mm_M4_ISO14580, MountingHole:MountingHole_4.3mm_M4_ISO14580, F.Cu at (150.5, 132.1)
Routing:
- net col6: track 172.8 -> 168.0 mm
- net col5: track 225.4 -> 222.1 mm
- net col4: track 242.6 -> 240.0 mm
- net row4: track 249.8 -> 252.3 mm
- net col0: track 279.4 -> 277.9 mm
- net col2: track 243.3 -> 242.0 mm
- net col3: track 252.8 -> 251.5 mm
- net col1: track 262.0 -> 260.7 mm
