File: splitkb.kicad_pcb (KiCad board)
At the start: 2 copper layers, 153 x 121.4 mm, 80 parts, among them J1 MJ-4PP-9, K1 KEYSW, SW1 SW_PUSH, SW10 SW_PUSH, SW11 SW_PUSH, SW12 SW_PUSH, SW13 SW_PUSH, SW14 SW_PUSH, SW15 SW_PUSH, SW16 SW_PUSH, SW17 SW_PUSH, SW18 SW_PUSH, SW19 SW_PUSH, SW2 SW_PUSH, SW20 SW_PUSH, SW21 SW_PUSH, SW22 SW_PUSH, SW23 SW_PUSH, SW24 SW_PUSH, SW25 SW_PUSH, SW26 SW_PUSH, SW27 SW_PUSH, SW28 SW_PUSH, SW29 SW_PUSH, SW3 SW_PUSH, SW30 SW_PUSH, SW31 SW_PUSH, SW32 SW_PUSH, SW4 SW_PUSH, SW5 SW_PUSH, SW6 SW_PUSH, SW7 SW_PUSH, SW8 SW_PUSH, SW9 SW_PUSH, U1 ProMicro

Commit message: test
Parts:
- removed  : LOGO, picture:katamaran (x2)
- removed  : MountingHole_2.2mm_M2, MountingHole:MountingHole_2.2mm_M2 (x11)
- D1, D10, D11, D12, D13, D14, D15, D16, D17, D18, D19, D2, D20, D21, D22, D23, D24, D25, D26, D27, D28, D29, D3, D30, D31, D32, D4, D5, D6, D7, D8, D9: footprint kbd:D3_TH_SMD -> Diode_SMD:D_SOD-323_HandSoldering; moved to B.Cu
- K1: footprint kbd:ResetSW -> random-keyboard-parts:SKQG-1155865
- U1: value ProMicro -> ATMEGA32U4; footprint kbd:ProMicro_v2 -> Package_QFP:LQFP-44_10x10mm_P0.8mm; moved to B.Cu
- moved D28 113.0 mm to (171.8, 49.1)
- moved D23 107.7 mm to (152.8, 46.1)
- moved U1 106.1 mm to (97.7, 123.2)
- moved D18 103.3 mm to (133.7, 43.1)
- moved D13 100.1 mm to (114.7, 40.1)
- moved D29 99.0 mm to (171.8, 68.2)
- moved D24 92.6 mm to (152.8, 65.1)
- moved D9 92.6 mm to (95.6, 43.1)
- moved D30 87.1 mm to (171.9, 87.2)
- moved D19 87.0 mm to (133.7, 62.1)
- moved D5 85.9 mm to (76.6, 46.1)
- moved K1 84.7 mm to (110.6, 118.6), turned to 180 degrees
- moved D1 83.7 mm to (57.5, 45.6)
- moved D14 82.7 mm to (114.6, 59.1)
- moved D25 79.1 mm to (152.7, 84.1)
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Connections:
- U1 pad 10: row3 -> Net-(U1-Pad10)
- U1 pad 11: row4 -> Net-(U1-Pad11)
- U1 pad 14: col6 -> Net-(U1-Pad14)
- U1 pad 15: col5 -> Net-(U1-Pad15)
- U1 pad 16: col4 -> Net-(U1-Pad16)
- U1 pad 17: col3 -> Net-(U1-Pad17)
- U1 pad 18: col2 -> Net-(U1-Pad18)
- U1 pad 19: col1 -> Net-(U1-Pad19)
- U1 pad 20: col0 -> Net-(U1-Pad20)
- U1 pad 21: VCC -> Net-(U1-Pad21)
- U1 pad 22: reset -> Net-(U1-Pad22)
- U1 pad 23: GND -> Net-(U1-Pad23)
- U1 pad 3: GND -> Net-(U1-Pad3)
- U1 pad 4: GND -> Net-(U1-Pad4)
- U1 pad 6: data -> Net-(U1-Pad6)
- U1 pad 7: row0 -> Net-(U1-Pad7)
- U1 pad 8: row1 -> Net-(U1-Pad8)
- U1 pad 9: row2 -> Net-(U1-Pad9)
Routing:
- net row3: track 253.3 -> 0.00 mm, vias 9 -> 0
- net row2: track 249.3 -> 0.00 mm, vias 9 -> 0
- net row1: track 245.4 -> 0.00 mm, vias 9 -> 0
- net row0: track 241.4 -> 0.00 mm, vias 9 -> 0
- net Net-(D28-Pad2): track 151.6 -> 13.4 mm
- net Net-(D23-Pad2): track 142.5 -> 13.4 mm
- net Net-(D18-Pad2): track 133.2 -> 13.4 mm
- net Net-(D29-Pad2): track 134.0 -> 16.6 mm
- net col5: track 332.7 -> 217.4 mm, vias 9 -> 6
- net Net-(D13-Pad2): track 123.7 -> 13.0 mm
- net Net-(D24-Pad2): track 124.9 -> 16.6 mm
- net Net-(D30-Pad2): track 113.3 -> 16.5 mm
- net Net-(D9-Pad2): track 109.3 -> 13.2 mm
- net Net-(D14-Pad2): track 106.5 -> 16.6 mm
- net col4: track 316.2 -> 226.4 mm, vias 9 -> 6
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Other:
- outline, holes or cut-outs redrawn
