File: splitkb.sch (KiCad schematic (older format))
At the start: 73 parts, among them J1 MJ-4PP-9, K1 KEYSW, SW1 SW_PUSH, SW10 SW_PUSH, SW11 SW_PUSH, SW12 SW_PUSH, SW13 SW_PUSH, SW14 SW_PUSH, SW15 SW_PUSH, SW16 SW_PUSH, SW17 SW_PUSH, SW18 SW_PUSH, SW19 SW_PUSH, SW2 SW_PUSH, SW20 SW_PUSH, SW21 SW_PUSH, SW22 SW_PUSH, SW23 SW_PUSH, SW24 SW_PUSH, SW25 SW_PUSH, SW26 SW_PUSH, SW27 SW_PUSH, SW28 SW_PUSH, SW29 SW_PUSH, SW3 SW_PUSH, SW30 SW_PUSH, SW31 SW_PUSH, SW32 SW_PUSH, SW33 SW_PUSH, SW34 SW_PUSH, SW35 SW_PUSH, SW4 SW_PUSH, SW5 SW_PUSH, SW6 SW_PUSH, SW7 SW_PUSH, SW8 SW_PUSH, SW9 SW_PUSH, U1 ProMicro

Commit message: new rev
Parts:
- removed D10, D15, D20, D5: D, keyboard_parts:D_SOD123_axial, symbol keyboard_parts:D
- removed J1: MJ-4PP-9, MJ-4PP-9:MJ-4PP-9, symbol MJ-4PP-9:MJ-4PP-9
- removed SW10, SW15, SW20, SW5: SW_PUSH, Button_Switch_Keyboard:SW_Cherry_MX_1.00u_PCB, symbol keyboard_parts:SW_PUSH
- removed U1: ProMicro, promicro:ProMicro, symbol promicro:ProMicro
- added D17: D, kbd:D3_TH_SMD, symbol keyboard_parts:D
- added J1: MJ-4PP-9, kbd:MJ-4PP-9, symbol kbd:MJ-4PP-9
- added SW17: SW_PUSH, kbd:CherryMX_Choc_Hotswap, symbol keyboard_parts:SW_PUSH
- added U1: ProMicro, kbd:ProMicro_v2, symbol kbd:ProMicro
- D1, D2, D3, D4: footprint keyboard_parts:D_SOD123_axial -> kbd:D3_TH_SMD
- D10: renamed from D12; footprint keyboard_parts:D_SOD123_axial -> kbd:D3_TH_SMD
- D11: renamed from D13; footprint keyboard_parts:D_SOD123_axial -> kbd:D3_TH_SMD
- D12: renamed from D14; footprint keyboard_parts:D_SOD123_axial -> kbd:D3_TH_SMD
- D13: renamed from D16; footprint keyboard_parts:D_SOD123_axial -> kbd:D3_TH_SMD
- D14: renamed from D17; footprint keyboard_parts:D_SOD123_axial -> kbd:D3_TH_SMD
- D15: renamed from D18; footprint keyboard_parts:D_SOD123_axial -> kbd:D3_TH_SMD
- D16: renamed from D19; footprint keyboard_parts:D_SOD123_axial -> kbd:D3_TH_SMD
- D18: renamed from D21; footprint keyboard_parts:D_SOD123_axial -> kbd:D3_TH_SMD
- D19: renamed from D22; footprint keyboard_parts:D_SOD123_axial -> kbd:D3_TH_SMD
- D20: renamed from D23; footprint keyboard_parts:D_SOD123_axial -> kbd:D3_TH_SMD
- D21: renamed from D24; footprint keyboard_parts:D_SOD123_axial -> kbd:D3_TH_SMD
- D22: renamed from D25; footprint keyboard_parts:D_SOD123_axial -> kbd:D3_TH_SMD
- D23: renamed from D26; footprint keyboard_parts:D_SOD123_axial -> kbd:D3_TH_SMD
- D24: renamed from D27; footprint keyboard_parts:D_SOD123_axial -> kbd:D3_TH_SMD
- D25: renamed from D28; footprint keyboard_parts:D_SOD123_axial -> kbd:D3_TH_SMD
- D26: renamed from D29; footprint keyboard_parts:D_SOD123_axial -> kbd:D3_TH_SMD
- D27: renamed from D30; footprint keyboard_parts:D_SOD123_axial -> kbd:D3_TH_SMD
- D28: renamed from D31; footprint keyboard_parts:D_SOD123_axial -> kbd:D3_TH_SMD
- D29: renamed from D32; footprint keyboard_parts:D_SOD123_axial -> kbd:D3_TH_SMD
- D30: renamed from D33; footprint keyboard_parts:D_SOD123_axial -> kbd:D3_TH_SMD
- D31: renamed from D34; footprint keyboard_parts:D_SOD123_axial -> kbd:D3_TH_SMD
- D32: renamed from D35; footprint keyboard_parts:D_SOD123_axial -> kbd:D3_TH_SMD
- D5: renamed from D6; footprint keyboard_parts:D_SOD123_axial -> kbd:D3_TH_SMD
- D6: renamed from D7; footprint keyboard_parts:D_SOD123_axial -> kbd:D3_TH_SMD
- D7: renamed from D8; footprint keyboard_parts:D_SOD123_axial -> kbd:D3_TH_SMD
- D8: renamed from D9; footprint keyboard_parts:D_SOD123_axial -> kbd:D3_TH_SMD
- D9: renamed from D11; footprint keyboard_parts:D_SOD123_axial -> kbd:D3_TH_SMD
- K1: footprint keyboard_parts:SW_TACT_TH_HORIZ_LOW -> kbd:ResetSW
- SW1, SW2, SW3, SW4: footprint Button_Switch_Keyboard:SW_Cherry_MX_1.00u_PCB -> kbd:CherryMX_Hotswap
- SW10: renamed from SW12; footprint Button_Switch_Keyboard:SW_Cherry_MX_1.00u_PCB -> kbd:CherryMX_Hotswap
- SW11: renamed from SW13; footprint Button_Switch_Keyboard:SW_Cherry_MX_1.00u_PCB -> kbd:CherryMX_Hotswap
- SW12: renamed from SW14; footprint Button_Switch_Keyboard:SW_Cherry_MX_1.00u_PCB -> kbd:CherryMX_Hotswap
- SW13: renamed from SW16; footprint Button_Switch_Keyboard:SW_Cherry_MX_1.00u_PCB -> kbd:CherryMX_Hotswap
- SW14: renamed from SW17; footprint Button_Switch_Keyboard:SW_Cherry_MX_1.00u_PCB -> kbd:CherryMX_Hotswap
- SW15: renamed from SW18; footprint Button_Switch_Keyboard:SW_Cherry_MX_1.00u_PCB -> kbd:CherryMX_Hotswap
- SW16: renamed from SW19; footprint Button_Switch_Keyboard:SW_Cherry_MX_1.00u_PCB -> kbd:CherryMX_Hotswap
- SW18: renamed from SW21; footprint Button_Switch_Keyboard:SW_Cherry_MX_1.00u_PCB -> kbd:CherryMX_Hotswap
- SW19: renamed from SW22; footprint Button_Switch_Keyboard:SW_Cherry_MX_1.00u_PCB -> kbd:CherryMX_Hotswap
- SW20: renamed from SW23; footprint Button_Switch_Keyboard:SW_Cherry_MX_1.00u_PCB -> kbd:CherryMX_Hotswap
- SW21: renamed from SW24; footprint Button_Switch_Keyboard:SW_Cherry_MX_1.00u_PCB -> kbd:CherryMX_Hotswap
- SW22: renamed from SW25; footprint Button_Switch_Keyboard:SW_Cherry_MX_1.00u_PCB -> kbd:CherryMX_Choc_Hotswap
- SW23: renamed from SW26; footprint Button_Switch_Keyboard:SW_Cherry_MX_1.00u_PCB -> kbd:CherryMX_Hotswap
- SW24: renamed from SW27; footprint Button_Switch_Keyboard:SW_Cherry_MX_1.00u_PCB -> kbd:CherryMX_Hotswap
- SW25: renamed from SW28; footprint Button_Switch_Keyboard:SW_Cherry_MX_1.00u_PCB -> kbd:CherryMX_Hotswap
- SW26: renamed from SW29; footprint Button_Switch_Keyboard:SW_Cherry_MX_1.00u_PCB -> kbd:CherryMX_Hotswap
- SW27: renamed from SW30; footprint Button_Switch_Keyboard:SW_Cherry_MX_1.00u_PCB -> kbd:CherryMX_Choc_Hotswap
- SW28: renamed from SW31; footprint Button_Switch_Keyboard:SW_Cherry_MX_1.00u_PCB -> kbd:CherryMX_Hotswap
- SW29: renamed from SW32; footprint Button_Switch_Keyboard:SW_Cherry_MX_1.00u_PCB -> kbd:CherryMX_Hotswap
- SW30: renamed from SW33; footprint Button_Switch_Keyboard:SW_Cherry_MX_1.00u_PCB -> kbd:CherryMX_Hotswap
- SW31: renamed from SW34; footprint Button_Switch_Keyboard:SW_Cherry_MX_1.00u_PCB -> kbd:CherryMX_Hotswap
- SW32: renamed from SW35; footprint Button_Switch_Keyboard:SW_Cherry_MX_1.00u_PCB -> kbd:CherryMX_Hotswap
- SW5: renamed from SW6; footprint Button_Switch_Keyboard:SW_Cherry_MX_1.00u_PCB -> kbd:CherryMX_Hotswap
- SW6: renamed from SW7; footprint Button_Switch_Keyboard:SW_Cherry_MX_1.00u_PCB -> kbd:CherryMX_Hotswap
- SW7: renamed from SW8; footprint Button_Switch_Keyboard:SW_Cherry_MX_1.00u_PCB -> kbd:CherryMX_Hotswap
- SW8: renamed from SW9; footprint Button_Switch_Keyboard:SW_Cherry_MX_1.00u_PCB -> kbd:CherryMX_Hotswap
- SW9: renamed from SW11; footprint Button_Switch_Keyboard:SW_Cherry_MX_1.00u_PCB -> kbd:CherryMX_Hotswap
Connections:
- net GND: now also K1.2, J1.C, U1.23 (GND), U1.3 (GND), U1.4 (GND); no longer K1.1
- net VCC: now also J1.D, U1.21 (VCC)
- net col0: now also U1.20 (F4/A3)
- net col1: now also U1.19 (F5/A2)
- net col2: now also U1.18 (F6/A1)
- net col3: now also SW17.1, U1.17 (F7/A0)
- net col4: now also U1.16 (B1/15)
- net col5: now also U1.15 (B3/14)
- net col6: now also U1.14 (B2/16)
- net data: now also J1.B, U1.6 (3/D0/SCL)
- net reset: now also K1.1, U1.22 (RST); no longer K1.2
- net row0: now also U1.7 (4/D4)
- net row1: now also U1.8 (5/C6)
- net row2: now also U1.9 (6/D7)
- net row3: now also U1.10 (7/E6)
- net row4: now also D17.1, U1.11 (8/B4)
- new net: D17.2, SW17.2
- no-connect marks 8 -> 7
Other:
- moved on the sheet: K1

Commit message: minor adjustments
Connections:
- net GND: now also J1.B; no longer J1.C
- net VCC: now also J1.A; no longer J1.D
- net data: now also J1.C; no longer J1.B
Changed lines of the file:
@@
 L power:VCC #PWR0105
 U 1 1 5EFE2D39
-P 1685 905
-F 0 "#PWR0105" H 1685 755 50  0001 C CNN
-F 1 "VCC" H 1702 1078 50  0000 C CNN
-F 2 "" H 1685 905 50  0001 C CNN
-F 3 "" H 1685 905 50  0001 C CNN
-	1    1685 905
+P 1685 855
+F 0 "#PWR0105" H 1685 705 50  0001 C CNN
+F 1 "VCC" H 1702 1028 50  0000 C CNN
+F 2 "" H 1685 855 50  0001 C CNN
+F 3 "" H 1685 855 50  0001 C CNN
+	1    1685 855
 	1    0    0    -1
 $EndComp
@@
 L power:GND #PWR0103
 U 1 1 5EFDC487
-P 1665 1315
-F 0 "#PWR0103" H 1665 1065 50  0001 C CNN
-F 1 "GND" H 1670 1142 50  0000 C CNN
-F 2 "" H 1665 1315 50  0001 C CNN
-F 3 "" H 1665 1315 50  0001 C CNN
-	1    1665 1315
-	1    0    0    -1
-$EndComp
-Wire Wire Line
-	1275 1200 2085 1200
-Text GLabel 2085 1200 2    50   Input ~ 0
+P 1665 1365
+F 0 "#PWR0103" H 1665 1115 50  0001 C CNN
+F 1 "GND" H 1670 1192 50  0000 C CNN
+F 2 "" H 1665 1365 50  0001 C CNN
+F 3 "" H 1665 1365 50  0001 C CNN
+	1    1665 1365
+	1    0    0    -1
+$EndComp
+Wire Wire Line
+	1275 1200 1665 1200
+Text GLabel 2085 1150 2    50   Input ~ 0
 data
 $Comp
@@
 	1    0    0    -1
 $EndComp
-NoConn ~ 1275 1050
-Wire Wire Line
-	1275 1100 1685 1100
-Wire Wire Line
-	1685 1100 1685 905
-Wire Wire Line
-	1275 1150 1665 1150
-Wire Wire Line
-	1665 1150 1665 1315
+NoConn ~ 1275 1100
+Wire Wire Line
+	1275 1050 1685 1050
+Wire Wire Line
+	1685 1050 1685 855
 Connection ~ 10600 3200
 Wire Wire Line
@@
 	1    0    0    -1
 $EndComp
+Wire Wire Line
+	1665 1200 1665 1365
+Wire Wire Line
+	1275 1150 2085 1150
 $EndSCHEMATC

Commit message: test
Parts:
- removed U1: ProMicro, kbd:ProMicro_v2, symbol kbd:ProMicro
- added U1: ATMEGA32U4, Package_QFP:LQFP-44_10x10mm_P0.8mm, symbol keyboard_parts:ATMEGA32U4
- D1, D10, D11, D12, D13, D14, D15, D16, D17, D18, D19, D2, D20, D21, D22, D23, D24, D25, D26, D27, D28, D29, D3, D30, D31, D32, D4, D5, D6, D7, D8, D9: footprint kbd:D3_TH_SMD -> Diode_SMD:D_SOD-323_HandSoldering
- J1: footprint kbd:MJ-4PP-9 -> (none)
- K1: footprint kbd:ResetSW -> random-keyboard-parts:SKQG-1155865
Connections:
- no-connect marks 7 -> 1
