File: Left/stm32split.kicad_pcb (KiCad board)
At the start: 2 copper layers, 152.4 x 110.7 mm, 92 parts, among them J1 Conn_01x04, SW1 SW_Push, SW10 SW_Push, SW11 SW_Push, SW12 SW_Push, SW13 SW_Push, SW14 SW_Push, SW15 SW_Push, SW16 SW_Push, SW17 SW_Push, SW18 SW_Push, SW19 SW_Push, SW2 SW_Push, SW20 SW_Push, SW21 SW_Push, SW22 SW_Push, SW23 SW_Push, SW24 SW_Push, SW25 SW_Push, SW26 SW_Push, SW27 SW_Push, SW28 SW_Push, SW29 SW_Push, SW3 SW_Push, SW30 SW_Push, SW31 SW_Push, SW4 SW_Push, SW5 SW_Push, SW6 SW_Push, SW7 SW_Push, SW8 SW_Push, SW9 SW_Push, U1 SRV05-4, U2 STM32F103CBTx, U3 XC6206PxxxMR, Y1 8MHz

Commit message: changed vbus pin
Connections:
- J1 pad 1: Net-(J1-Pad1) -> GND
- J1 pad 2: VBUS -> SPLITHANDPIN
- J1 pad 3: SPLITHANDPIN -> (no net)
- J1 pad 4: GND -> VBUS
Routing:
- net VBUS: track 31.2 -> 26.8 mm
- net SPLITHANDPIN: track 30.1 -> 34.1 mm
Changed lines of the file:
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@@
     (thickness 1.6)
     (drawings 251)
-    (tracks 3844)
+    (tracks 3847)
     (zones 0)
     (modules 92)
-    (nets 82)
+    (nets 81)
   )
   (page A4)
@@
     (mod_text_size 1 1)
     (mod_text_width 0.15)
-    (pad_size 1.524 1.524)
-    (pad_drill 0.762)
+    (pad_size 1.8 1.2)
+    (pad_drill 1.2)
     (pad_to_mask_clearance 0.051)
     (solder_mask_min_width 0.25)
@@
   (net 79 SOFTSERIALPIN)
   (net 80 SPLITHANDPIN)
-  (net 81 "Net-(J1-Pad1)")
   (net_class Default "This is the default net class."
     (clearance 0.2)
@@
     (add_net "Net-(D8-Pad2)")
     (add_net "Net-(D9-Pad2)")
-    (add_net "Net-(J1-Pad1)")
     (add_net "Net-(R1-Pad2)")
     (add_net "Net-(R2-Pad2)")
@@
     (pad "" np_thru_hole circle (at 1.6 0 270) (size 1.5 1.5) (drill 1.5) (layers *.Cu *.Mask))
     (pad 4 thru_hole oval (at 11.3 2.3 270) (size 1.8 1.2) (drill oval 1.2 0.6) (layers *.Cu *.Mask)
-      (net 66 GND))
-    (pad 3 thru_hole oval (at 10.2 -2.3 270) (size 1.8 1.2) (drill oval 1.2 0.6) (layers *.Cu *.Mask)
-      (net 80 SPLITHANDPIN))
-    (pad 2 thru_hole oval (at 6.2 -2.3 270) (size 1.8 1.2) (drill oval 1.2 0.6) (layers *.Cu *.Mask)
       (net 65 VBUS))
+    (pad 3 thru_hole oval (at 10.2 -2.3 270) (size 1.8 1.2) (drill oval 1.2 0.6) (layers *.Cu *.Mask))
+    (pad 2 thru_hole oval (at 6.2 -2.3 270) (size 1.8 1.2) (drill oval 1.2 0.6) (layers *.Cu *.Mask)
+      (net 80 SPLITHANDPIN))
     (pad 1 thru_hole oval (at 3.2 -2.3 270) (size 1.8 1.2) (drill oval 1.2 0.6) (layers *.Cu *.Mask)
-      (net 81 "Net-(J1-Pad1)"))
+      (net 66 GND))
   )
   (module Crystal:Crystal_SMD_5032-2Pin_5.0x3.2mm (layer F.Cu)
@@
   (segment (start 188.84375 88.24625) (end 188.83 88.26) (width 0.5) (layer F.Cu) (net 65))
   (via (at 188.83 88.26) (size 0.8) (drill 0.4) (layers F.Cu B.Cu) (net 65))
-  (segment (start 193.74 88.26) (end 200.03 88.26) (width 0.5) (layer F.Cu) (net 65))
-  (segment (start 202.41 85.88) (end 204.70625 85.88) (width 0.5) (layer F.Cu) (net 65))
-  (segment (start 200.03 88.26) (end 202.41 85.88) (width 0.5) (layer F.Cu) (net 65))
+  (segment (start 194.305685 88.26) (end 193.74 88.26) (width 0.5) (layer F.Cu) (net 65))
+  (segment (start 196.28625 88.26) (end 194.305685 88.26) (width 0.5) (layer F.Cu) (net 65))
+  (segment (start 199.00625 90.98) (end 196.28625 88.26) (width 0.5) (layer F.Cu) (net 65))
+  (segment (start 200.10625 90.98) (end 199.00625 90.98) (width 0.5) (layer F.Cu) (net 65))
   (segment (start 188.06875 85.9825) (end 188.06875 85.6625) (width 0.3) (layer F.Cu) (net 66))
   (segment (start 188.06875 85.6625) (end 186.97375 84.5675) (width 0.3) (layer F.Cu) (net 66))
@@
   (segment (start 195.62375 111.75625) (end 196.43 110.95) (width 0.3) (layer F.Cu) (net 80))
   (segment (start 191.11625 111.75625) (end 195.62375 111.75625) (width 0.3) (layer F.Cu) (net 80))
-  (segment (start 204.70625 102.67375) (end 204.70625 89.88) (width 0.25) (layer B.Cu) (net 80))
-  (segment (start 196.43 110.95) (end 204.70625 102.67375) (width 0.25) (layer B.Cu) (net 80))
+  (segment (start 204.70625 87.03) (end 204.70625 85.88) (width 0.25) (layer B.Cu) (net 80))
+  (segment (start 203.481251 88.254999) (end 204.70625 87.03) (width 0.25) (layer B.Cu) (net 80))
+  (segment (start 203.481251 103.898749) (end 203.481251 88.254999) (width 0.25) (layer B.Cu) (net 80))
+  (segment (start 196.43 110.95) (end 203.481251 103.898749) (width 0.25) (layer B.Cu) (net 80))
   (zone (net 66) (net_name GND) (layer F.Cu) (hatch edge 0.508)
     (connect_pads (clearance 0.508))
